Commit message: Finally!!! Sensor detects rope

File: gymnasium_env/envs/pybullet_ur5_gripper/robots/urdf/ur5e_with_gripper_digit.urdf (robot description, URDF)
Before this commit: robot ur5e_gripper, 21 links, 20 joints
Joints:
- joint sensor_gripper_joint: origin xyz=0.2 0.0 0.0 rpy=0.0 0.0 1.5708 -> xyz=0.01 -0.01 0.0 rpy=1.5708 0.0 1.5708

Commit message: new position of sensor in urdf

File: gymnasium_env/envs/pybullet_ur5_gripper/robots/urdf/ur5e_with_gripper_digit.urdf (robot description, URDF)
Before this commit: robot ur5e_gripper, 21 links, 20 joints
Joints:
- joint sensor_gripper_joint: origin xyz=0.01 -0.01 0.0 rpy=1.5708 0.0 1.5708 -> xyz=0.004 -0.009 0.0 rpy=1.5708 0.0 1.5708

Commit message: new lowfreq env

File: gymnasium_env/envs/pybullet_ur5_gripper/robots/urdf/ur5e_with_gripper_digit.urdf (robot description, URDF)
Before this commit: robot ur5e_gripper, 21 links, 20 joints
Joints:
- joint sensor_gripper_joint: origin xyz=0.004 -0.009 0.0 rpy=1.5708 0.0 1.5708 -> xyz=0.01 -0.01 0.0 rpy=1.5708 0.0 1.5708
